File: bacee/Connectors.sch (KiCad schematic (older format))
At the start: 4 parts, among them J1 ICSP, J2 Digital Pins, J3 Serial Port, J4 I2C

Commit message: wip: wiring
Connections:
- net D2: now reaches J2.1 (Pin_1)
- net D3: now reaches J2.2 (Pin_2)
- net D4: now reaches J2.3 (Pin_3)
- net D5: now reaches J2.4 (Pin_4)
- net D6: now reaches J2.5 (Pin_5)
- net D7: now reaches J2.6 (Pin_6)
- net D8: now reaches J2.7 (Pin_7)
- net GND: now reaches J2.8 (Pin_8)
- net GND: now also J1.6 (Pin_6), J3.1 (Pin_1), J4.1 (Pin_1)
- net VCC: now reaches J2.9 (Pin_9)
- net VCC: now also J1.2 (Pin_2), J3.2 (Pin_2), J4.2 (Pin_2)
- net RX: now reaches J3.3 (Pin_3)
- net TX: now reaches J3.4 (Pin_4)
- net MISO: now reaches J1.1 (Pin_1)
- net SCK: now reaches J1.3 (Pin_3)
- net SCK: now also J4.4 (Pin_4)
- net MOSI: now reaches J1.4 (Pin_4)
- net RESET: now reaches J1.5 (Pin_5)
- net SDA: now reaches J4.3 (Pin_3)
Changed lines of the file:
@@
 	1    0    0    -1
 $EndComp
+Text HLabel 4300 4250 0    50   Output ~ 0
+MISO
+Text HLabel 4300 4350 0    50   BiDi ~ 0
+SCK
+Text HLabel 4300 4450 0    50   Output ~ 0
+RESET
+Text HLabel 4800 4250 2    50   Input ~ 0
+VCC
+Text HLabel 4800 4350 2    50   Input ~ 0
+MOSI
+Text HLabel 4800 4450 2    50   Input ~ 0
+GND
+Text HLabel 5800 2950 0    50   Input ~ 0
+GND
+Text HLabel 5800 3050 0    50   Input ~ 0
+VCC
+Text HLabel 5800 3150 0    50   Input ~ 0
+RX
+Text HLabel 5800 3250 0    50   Output ~ 0
+TX
+Text HLabel 5800 4100 0    50   Input ~ 0
+GND
+Text HLabel 5800 4200 0    50   Input ~ 0
+VCC
+Text HLabel 5800 4300 0    50   BiDi ~ 0
+SDA
+Text HLabel 5800 4400 0    50   BiDi ~ 0
+SCK
+Text HLabel 4350 2650 0    50   BiDi ~ 0
+D2
+Text HLabel 4350 2750 0    50   BiDi ~ 0
+D3
+Text HLabel 4350 2850 0    50   BiDi ~ 0
+D4
+Text HLabel 4350 2950 0    50   BiDi ~ 0
+D5
+Text HLabel 4350 3050 0    50   BiDi ~ 0
+D6
+Text HLabel 4350 3150 0    50   BiDi ~ 0
+D7
+Text HLabel 4350 3250 0    50   BiDi ~ 0
+D8
+Text HLabel 4350 3350 0    50   Input ~ 0
+GND
+Text HLabel 4350 3450 0    50   Input ~ 0
+VCC
 $EndSCHEMATC
