File: bacee/bacee.sch (KiCad schematic (older format))
At the start: 13 parts, among them U1 24LC1025, U2 24LC1025, U3 DS13375+, U4 ATMEGA328P-AU, Y1 Crystal 32MHz, Y2 Crystal 16MHz

Commit message: wip: wiring
Connections:
- net GND: now also U1.2 (A1), U1.4 (GND), U1.7 (WP), U2.2 (A1), U2.4 (GND), U2.7 (WP), U3.4 (GND), U4.21 (GND), U4.3 (GND), U4.5 (GND)
- net VCC: now reaches U1.1 (A0)
- net VCC: now also U1.3 (A2), U1.8 (VCC), U2.1 (A0), U2.3 (A2), U2.8 (VCC), U4.18 (AVCC), U4.4 (VCC), U4.6 (VCC)
- net SDA: now reaches U1.5 (SDA)
- net SDA: now also U2.5 (SDA), U4.27 (PC4)
- net SCL: now reaches U1.6 (SCL)
- net SCL: now also U2.6 (SCL), U4.28 (PC5)
- net D3: now reaches U4.1 (PD3)
- net D6: now reaches U4.10 (PD6)
- net D7: now reaches U4.11 (PD7)
- net D8: now reaches U4.12 (PB0)
- net MOSI: now reaches U4.15 (PB3)
- net MISO: now reaches U4.16 (PB4)
- net SCK: now reaches U4.17 (PB5)
- net D4: now reaches U4.2 (PD4)
- net RESET: now reaches U4.29 (PC6)
- net RX: now reaches U4.30 (PD0)
- net TX: now reaches U4.31 (PD1)
- net D2: now reaches U4.32 (PD2)
- net D5: now reaches U4.9 (PD5)
- net at U3.1 (X1): now also Y1.1
- net at U3.2 (X2): now also Y1.2
Other:
- moved on the sheet: U1, U2, Y1

Commit message: done
Parts:
- Y1: value Crystal 32MHz -> Crystal 32768 kHz
Connections:
- net GND is gone; now on net GNDPWR: U1.2 (A1), U1.4 (GND), U1.7 (WP), U2.2 (A1), U2.4 (GND), U2.7 (WP), U3.4 (GND), U4.21 (GND), U4.3 (GND), U4.5 (GND)
- net RESET: now also R2.1
- net SCK: now also D1.2 (A), U3.6 (SCL)
- net SDA: now also U3.5 (SDA)
- net VCC: now also BT1.1 (+), C3.1, R2.2, U3.3 (INTA), U3.8 (Vcc), U4.20 (AREF)
- net GNDPWR: now reaches BT1.2 (-)
- net GNDPWR: now also C1.2, C2.2, C3.2, R1.2
- net at C1.1: now also U4.7 (PB6), Y2.1
- net at C2.1: now also U4.8 (PB7), Y2.2
- net at D1.1 (K): now also R1.1
- no-connect marks 0 -> 9
Other:
- moved on the sheet: BT1, C1, C2, C3, D1, R1, R2, U3, Y1
