File: bacee/bacee_2_layer_kicad_pcb.kicad_pcb (KiCad board)
At the start: 2 copper layers, 38.1 x 29.2 mm, 17 parts, among them J1 ICSP, J2 Digital Pins, J3 Serial Port, J4 I2C, U1 24LC1025, U2 24LC1025, U3 DS13375+, U4 ATMEGA328P-AU, Y1 Crystal 32768 kHz, Y2 Crystal 16MHz

Commit message: done
Routing:
- removed copper zone on B.Cu, net GNDPWR
